File: can-bus.kicad_sch (KiCad schematic)
At the start: 12 parts, among them P3 TERM, P4 TERM, U9 IFX1050GVIOXUMA1

Commit message: Finalized project
Parts:
- removed D2, D3, D4: SMAJ18CA, Diodes:SMAJ18CA_SMD_DO214AC, symbol Diodes:SMAJ18CA
- added D2: PESD2CAN, ESD_Protectors:PESD2CAN.215, symbol esd_protectors:PESD2CAN
Connections:
- net GND: now also D2.3 (GND)
- net at F2.1, P4.1, U9.6 (CANL): now also D2.1 (I/O1)
- net at F1.1, P3.2, U9.7 (CANH): now also D2.2 (I/O2)
Other:
- moved on the sheet: F1, F2
